File: PCB/PCB-backups/PCB-2026-06-28_135803/PCB.kicad_sch (KiCad schematic)
At the start: 5 parts, among them SW1 SW_Wuerth_450301014042, U1 XIAO-ESP32-S3-SMD, U3 adafruit-MAX98357

Commit message: Changed Silkscreen, PCB Up To Date
Parts:
- added R2: 100 kOhms, Resistor_SMD:R_0805_2012Metric, symbol Device:R
Connections:
- net GND: now also R2.2; no longer U1.25 (PAD), U3.4 (GAIN)
- new net: R2.1, U3.4 (GAIN)
- no-connect marks 18 -> 12
Changed lines of the file:
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@@
 	(paper "A4")
 	(no_connect
-		(at 130.81 86.36)
-	)
-	(no_connect
 		(at 166.37 106.68)
 	)
 	(no_connect
-		(at 149.86 86.36)
-	)
-	(no_connect
-		(at 138.43 86.36)
-	)
-	(no_connect
 		(at 123.19 102.87)
 	)
@@
 	)
 	(no_connect
-		(at 146.05 86.36)
-	)
-	(no_connect
 		(at 123.19 99.06)
 	)
@@
 	)
 	(no_connect
-		(at 157.48 86.36)
-	)
-	(no_connect
 		(at 166.37 99.06)
 	)
 	(no_connect
-		(at 153.67 86.36)
-	)
-	(no_connect
 		(at 166.37 114.3)
 	)
@@
 	)
 	(no_connect
-		(at 134.62 86.36)
+		(at 149.86 130.81)
 	)
 	(no_connect
@@
 	(wire
 		(pts
-			(xy 157.48 63.5) (xy 157.48 64.77)
+			(xy 157.48 64.77) (xy 132.08 64.77)
 		)
 		(stroke
@@
 	(wire
 		(pts
-			(xy 157.48 63.5) (xy 132.08 63.5)
+			(xy 132.08 64.77) (xy 132.08 68.58)
 		)
 		(stroke
@@
 	(wire
 		(pts
-			(xy 132.08 63.5) (xy 132.08 68.58)
+			(xy 232.41 76.2) (xy 232.41 78.74)
 		)
 		(stroke
@@
 		)
 	)
-	(wire
-		(pts
-			(xy 232.41 76.2) (xy 232.41 78.74)
-		)
-		(stroke
-			(width 0)
-			(type default)
-		)
-	)
 	(global_label "D8"
 		(shape input)
@@
 				)
 				(justify left)
-			)
-		)
-	)
-	(global_label "GND"
-		(shape input)
-		(at 232.41 91.44 0)
-		(fields_autoplaced yes)
-		(effects
-			(font
-				(size 1.27 1.27)
-			)
-			(justify left)
-		)
-		(property "Intersheetrefs" "${INTERSHEET_REFS}"
-			(at 239.2657 91.44 0)
-			(hide yes)
-			(show_name no)
-			(do_not_autoplace no)
-			(effects
-				(font
-					(size 1.27 1.27)
-				)
-				(justify left)
-			)
-		)
-	)
-	(global_label "GND"
-		(shape input)
-		(at 149.86 130.81 270)
-		(fields_autoplaced yes)
-		(effects
-			(font
-				(size 1.27 1.27)
-			)
-			(justify right)
-		)
-		(property "Intersheetrefs" "${INTERSHEET_REFS}"
-			(at 149.86 137.6657 90)
-			(hide yes)
-			(show_name no)
-			(do_not_autoplace no)
-			(effects
-				(font
-					(size 1.27 1.27)
-				)
-				(justify right)
 			)
 		)
@@
 					(unit 1)
 				)
+			)
+		)
+	)
+	(symbol
+		(lib_id "Device:R")
+		(at 232.41 95.25 0)
+		(unit 1)
+		(body_style 1)
+		(exclude_from_sim no)
+		(in_bom yes)
+		(on_board yes)
+		(in_pos_files yes)
+		(dnp no)
+		(property "Reference" "R2"
+			(at 234.95 93.9799 0)
+			(show_name no)
+			(do_not_autoplace no)
+			(effects
+				(font
+					(size 1.27 1.27)
+				)
+				(justify left)
+			)
+		)
+		(property "Value" "100 kOhms"
+			(at 232.41 97.282 90)
+			(show_name no)
+			(do_not_autoplace no)
+			(effects
+				(font
+					(size 0.508 0.508)
+				)
+				(justify left)
+			)
+		)
+		(property "Footprint" "Resistor_SMD:R_0805_2012Metric"
+			(at 230.632 95.25 90)
+			(hide yes)
+			(show_name no)
+			(do_not_autoplace no)
+			(effects
+				(font
+					(size 1.27 1.27)
+				)
+			)
+		)
+		(property "Datasheet" ""
+			(at 232.41 95.25 0)
+			(hide yes)
+			(show_name no)
+			(do_not_autoplace no)
+			(effects
+				(font
+					(size 1.27 1.27)
+				)
+			)
+		)
+		(property "Description" "Resistor"
+			(at 232.41 95.25 0)
+			(hide yes)
+			(show_name no)
+			(do_not_autoplace no)
+			(effects
+				(font
+					(size 1.27 1.27)
+				)
+			)
+		)
+		(pin "1"
+		)
+		(pin "2"
+		)
+		(instances
+			(project "PCB"
+				(path "/3851a501-b3a0-4d0a-bb18-9db29ab625cd"
+					(reference "R2")
+					(unit 1)
+				)
+			)
+		)
+	)
+	(symbol
+		(lib_id "power:GND")
+		(at 232.41 99.06 0)
+		(unit 1)
+		(body_style 1)
+		(exclude_from_sim no)
+		(in_bom yes)
+		(on_board yes)
+		(in_pos_files yes)
+		(dnp no)
+		(fields_autoplaced yes)
+		(property "Reference" "#PWR02"
+			(at 232.41 105.41 0)
+			(hide yes)
+			(show_name no)
+			(do_not_autoplace no)
+			(effects
+				(font
+					(size 1.27 1.27)
+				)
+			)
+		)
+		(property "Value" "GND"
+			(at 232.41 104.14 0)
+			(show_name no)
+			(do_not_autoplace no)
+			(effects
+				(font
+					(size 1.27 1.27)
+				)
+			)
+		)
+		(property "Footprint" ""
+			(at 232.41 99.06 0)
+			(hide yes)
+			(show_name no)
+			(do_not_autoplace no)
+			(effects
+				(font
+					(size 1.27 1.27)
+				)
+			)
+		)
+		(property "Datasheet" ""
+			(at 232.41 99.06 0)
+			(hide yes)
+			(show_name no)
+			(do_not_autoplace no)
+			(effects
+				(font
+					(size 1.27 1.27)
+				)
+			)
+		)
+		(property "Description" "Power symbol creates a global label with name \"GND\" , ground"
+			(at 232.41 99.06 0)
+			(hide yes)
+			(show_name no)
+			(do_not_autoplace no)
+			(effects
+				(font
+					(size 1.27 1.27)
+				)
+			)
+		)
+		(pin "1"
+		)
+		(instances
+			(project "PCB"
+				(path "/3851a501-b3a0-4d0a-bb18-9db29ab625cd"
+					(reference "#PWR02")
+					(unit 1)
+				)
